File: full-wave-rectifier.kicad_sch (KiCad schematic)
At the start: 40 parts, among them J10 Control Right, J11 Main Right, J2 Input Ch1, J3 Input Ch2, J4 Output Ch1, J5 Output Ch2, J6 Ochd input, J8 Control Left, J9 Main Left, U2 TL074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

Commit message: save changes
Parts:
- D3, D4, D5, D6: footprint Diode_SMD:D_SOD-123 -> Eurorack:D_SOD-123_Metric1.30x1.75mm_HandSolder
Changed lines of the file:
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@@
 			)
 		)
-		(property "Footprint" "Diode_SMD:D_SOD-123"
+		(property "Footprint" "Eurorack:D_SOD-123_Metric1.30x1.75mm_HandSolder"
 			(at 130.175 121.92 0)
 			(effects
@@
 			)
 		)
-		(property "Footprint" "Diode_SMD:D_SOD-123"
+		(property "Footprint" "Eurorack:D_SOD-123_Metric1.30x1.75mm_HandSolder"
 			(at 128.905 57.15 0)
 			(effects
@@
 			)
 		)
-		(property "Footprint" "Diode_SMD:D_SOD-123"
+		(property "Footprint" "Eurorack:D_SOD-123_Metric1.30x1.75mm_HandSolder"
 			(at 114.3 130.175 0)
 			(effects
@@
 			)
 		)
-		(property "Footprint" "Diode_SMD:D_SOD-123"
+		(property "Footprint" "Eurorack:D_SOD-123_Metric1.30x1.75mm_HandSolder"
 			(at 113.03 65.405 0)
 			(effects
