File: full-wave-rectifier.kicad_pcb (KiCad board)
At the start: 2 copper layers, 80.6 x 108 mm, 65 parts, among them J10 Control Right, J11 Main Right, J12 Power Connector, J2 Input Ch1, J3 Input Ch2, J4 Output Ch1, J5 Output Ch2, J6 Ochd input, J8 Control Left, J9 Main Left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

Commit message: save chages
Parts:
- moved C1 2.20 mm to (173.7, 139.7)
Routing:
- net M_OUTPUT_CH1: track 14.1 -> 16.3 mm
- net M_OUTPUT_CH2: track 14.1 -> 16.3 mm
- net M_OFFSET_CH1: track 16.3 -> 15.6 mm
- net GND: vias 13 -> 14

Commit message: save changes
Parts:
- removed C15: 1uF, Capacitor_THT:C_Rect_L7.2mm_W4.5mm_P5.00mm_FKS2_FKP2_MKS2_MKP2
- removed C3, C4: 10uF, Capacitor_THT:CP_Radial_D5.0mm_P2.00mm
- removed C7, C8: 100nF, Capacitor_SMD:C_1206_3216Metric_Pad1.33x1.80mm_HandSolder
- removed R23: 100, Resistor_SMD:R_1206_3216Metric_Pad1.30x1.75mm_HandSolder
- removed U1: LM78L05_TO92, Package_TO_SOT_THT:TO-92_Inline_Wide
- added C16: 100nF, Capacitor_SMD:C_1206_3216Metric_Pad1.33x1.80mm_HandSolder, F.Cu at (234.5, 133.4)
- added D22: D_TVS, Diode_SMD:D_SOD-323_HandSoldering, F.Cu at (221.1, 128.5)
- added D23: D_TVS, Diode_SMD:D_SOD-323_HandSoldering, F.Cu at (221.1, 131.4)
- added D24: D_TVS, Diode_SMD:D_SOD-323_HandSoldering, F.Cu at (221.1, 134.4)
- added D25: D_TVS, Diode_SMD:D_SOD-323_HandSoldering, F.Cu at (221.1, 137.3)
- added F1: Polyfuse, Fuse:Fuse_1206_3216Metric_Pad1.42x1.75mm_HandSolder, F.Cu at (228.6, 128.7)
- added F2: Polyfuse, Fuse:Fuse_1206_3216Metric_Pad1.42x1.75mm_HandSolder, F.Cu at (228.6, 132.0)
- added R24: 3.3k, Resistor_SMD:R_1206_3216Metric_Pad1.30x1.75mm_HandSolder, F.Cu at (228.6, 135.3)
- added U5: LM4040DBZ-5, Package_TO_SOT_SMD:SOT-23_Handsoldering, F.Cu at (234.8, 129.5)
- C1, C2: value 10uF -> 22uF, 25V
Connections:
- J12 pad 1: Net-(Q7-D) -> Net-(F2-Pad1)
- J12 pad 10: Net-(Q8-D) -> Net-(F1-Pad1)
- J12 pad 2: Net-(Q7-D) -> Net-(F2-Pad1)
- J12 pad 9: Net-(Q8-D) -> Net-(F1-Pad1)
- J4 pad TN: GND -> unconnected-(J4-PadTN)
- J5 pad TN: GND -> unconnected-(J5-PadTN)
Routing:
- net +12V: track 116.8 -> 102.3 mm, vias 4 -> 3
- net Net-(U1-VO): track 12.1 -> 0.00 mm
- net +5V: track 23.6 -> 13.6 mm
