File: faceplate/faceplate.kicad_pcb (KiCad board)
At the start: 2 copper layers, 30 x 128.5 mm, 0 parts

Commit message: Added JLCJLCJLCJLC
Other:
- board text added: "JLCJLCJLCJLC"
Changed lines of the file:
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@@
 		(end 138.600005 46.309124)
 		(stroke
-			(width 0)
+			(width 0.1)
 			(type solid)
 		)
@@
 		(layer "Edge.Cuts")
 	)
+	(gr_text "JLCJLCJLCJLC"
+		(at 157.48 159.385 -0)
+		(layer "B.SilkS")
+		(effects
+			(font
+				(size 1 1)
+				(thickness 0.15)
+			)
+			(justify left bottom mirror)
+		)
+	)
 	(group ""
